File: PDBueno/BYTE_Electronics.kicad_sch (KiCad schematic)
At the start: 17 parts, among them J1 Battery 2, J2 Battery 1, J3 Battery Buck 24V, J4 Screw_Terminal_01x02, J5 Battery Buck 48V, J7 Screw_Terminal_01x02, J9 Screw_Terminal_01x02, SW1 SW_DPST_x2, U1 BEC_Matek

Commit message: PCB routing
Parts:
- removed SW1: SW_DPST_x2, symbol Switch:SW_DPST_x2
- removed TP_GND2: TestPoint, symbol Connector:TestPoint
- J3, J5: footprint (none) -> TerminalBlock:TerminalBlock_MaiXu_MX126-5.0-02P_1x02_P5.00mm
- TP+24V1: renamed from TP2; footprint (none) -> TestPoint:TestPoint_Pad_D4.0mm
- TP+48V1: renamed from TP1; footprint (none) -> TestPoint:TestPoint_Pad_D4.0mm
- TP_GND1: footprint (none) -> TestPoint:TestPoint_Pad_D4.0mm
- U1: value BEC_Matek -> Buck Converter
Connections:
- net Battery 1 + is gone; now on net +48V: TP+48V1.1
- net Battery 1 - is gone; now on net GND: TP_GND1.1
- net Battery 2 + is gone; now on net +24V: TP+24V1.1
- net +48V: now also J1.2 (Pin_2)
- net GND: now also J2.1 (Pin_1); no longer J1.2 (Pin_2)
- no-connect marks 1 -> 5
Other:
- note added: "Actuators power connection"
- note added: "Buck Connection"
- note added: "Test Points"
- note removed: "Back converter"
- note removed: "TP Battery 1"
- note removed: "TP Battery 2"
- company: (none) -> AI-Team
- title: (none) -> PDBueno
- moved on the sheet: R1, TP+24V1, TP+48V1, TP_GND1, U1
