File: PDBueno/PDBueno.kicad_sch (KiCad schematic)
At the start: 15 parts, among them J1 Battery 2, J2 Battery 1, J3 Battery Buck 24V, J4 Screw_Terminal_01x02, J5 Battery Buck 48V, J7 Screw_Terminal_01x02, J9 Screw_Terminal_01x02, U1 Buck Converter

Commit message: 50th copper pour
Parts:
- added H1, H2, H3, H4: MountingHole_Pad, MountingHole:MountingHole_3.2mm_M3_Pad_Via, symbol Mechanical:MountingHole_Pad
Connections:
- net GND: now also H1.1, H2.1, H3.1, H4.1

Commit message: updates updates updates...
Parts:
- J3, J5: footprint TerminalBlock:TerminalBlock_MaiXu_MX126-5.0-02P_1x02_P5.00mm -> TerminalBlock:TerminalBlock_bornier-2_P5.08mm
Connections:
- net +24V: now also J3.2 (Pin_2); no longer J3.1 (Pin_1)
- net +48V: now also J4.2 (Pin_2), J5.2 (Pin_2), J7.2 (Pin_2), J9.2 (Pin_2); no longer J4.1 (Pin_1), J5.1 (Pin_1), J7.1 (Pin_1), J9.1 (Pin_1)
- net GND: now also J3.1 (Pin_1), J4.1 (Pin_1), J5.1 (Pin_1), J7.1 (Pin_1), J9.1 (Pin_1); no longer J3.2 (Pin_2), J4.2 (Pin_2), J5.2 (Pin_2), J7.2 (Pin_2), J9.2 (Pin_2)
Other:
- note added: "Mounting Holes"
- moved on the sheet: C1, C2, C3
