File: PDBueno/PDBueno.kicad_pcb (KiCad board)
At the start: 2 copper layers, 129.5 x 81.3 mm, 19 parts, among them J1 Battery 2, J2 Battery 1, J3 Battery Buck 24V, J4 Screw_Terminal_01x02, J5 Battery Buck 48V, J7 Screw_Terminal_01x02, J9 Screw_Terminal_01x02, U1 Buck Converter

Commit message: Added vias to properly connect capacitors to GND
Parts:
- moved U1 2.54 mm to (142.2, 94.0)
Routing:
- net GND: track 10.7 -> 57.8 mm, vias 2 -> 5
Other:
- board text added: "+"
- board text added: "-"
Changed lines of the file:
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@@
 		(property ki_fp_filters "TerminalBlock*:*")
 		(sheetname "/")
-		(sheetfile "BYTE_Electronics.kicad_sch")
+		(sheetfile "PDBueno.kicad_sch")
 		(attr through_hole)
 		(fp_line
@@
 		(property ki_fp_filters "CP_*")
 		(sheetname "/")
-		(sheetfile "BYTE_Electronics.kicad_sch")
+		(sheetfile "PDBueno.kicad_sch")
 		(attr smd)
 		(fp_line
@@
 		(property ki_fp_filters "CP_*")
 		(sheetname "/")
-		(sheetfile "BYTE_Electronics.kicad_sch")
+		(sheetfile "PDBueno.kicad_sch")
 		(attr smd)
 		(fp_line
@@
 		(property ki_fp_filters "CP_*")
 		(sheetname "/")
-		(sheetfile "BYTE_Electronics.kicad_sch")
+		(sheetfile "PDBueno.kicad_sch")
 		(attr smd)
 		(fp_line
@@
 		(property ki_fp_filters "Pin* Test*")
 		(sheetname "/")
-		(sheetfile "BYTE_Electronics.kicad_sch")
+		(sheetfile "PDBueno.kicad_sch")
 		(attr exclude_from_pos_files)
 		(fp_circle
@@
 		(property ki_fp_filters "TerminalBlock*:*")
 		(sheetname "/")
-		(sheetfile "BYTE_Electronics.kicad_sch")
+		(sheetfile "PDBueno.kicad_sch")
 		(attr through_hole)
 		(fp_line
@@
 		(property ki_fp_filters "TerminalBlock*:*")
 		(sheetname "/")
-		(sheetfile "BYTE_Electronics.kicad_sch")
+		(sheetfile "PDBueno.kicad_sch")
 		(attr through_hole)
 		(fp_line
@@
 		(property ki_fp_filters "TerminalBlock*:*")
 		(sheetname "/")
-		(sheetfile "BYTE_Electronics.kicad_sch")
+		(sheetfile "PDBueno.kicad_sch")
 		(attr through_hole)
 		(fp_line
@@
 		(property ki_fp_filters "TerminalBlock*:*")
 		(sheetname "/")
-		(sheetfile "BYTE_Electronics.kicad_sch")
+		(sheetfile "PDBueno.kicad_sch")
 		(attr through_hole)
 		(fp_line
@@
 		(property ki_fp_filters "TerminalBlock*:*")
 		(sheetname "/")
-		(sheetfile "BYTE_Electronics.kicad_sch")
+		(sheetfile "PDBueno.kicad_sch")
 		(attr through_hole)
 		(fp_line
@@
 		(property ki_fp_filters "Pin* Test*")
 		(sheetname "/")
-		(sheetfile "BYTE_Electronics.kicad_sch")
+		(sheetfile "PDBueno.kicad_sch")
 		(attr exclude_from_pos_files)
 		(fp_circle
@@
 		(property ki_fp_filters "Pin* Test*")
 		(sheetname "/")
-		(sheetfile "BYTE_Electronics.kicad_sch")
+		(sheetfile "PDBueno.kicad_sch")
 		(attr exclude_from_pos_files)
 		(fp_circle
@@
 		(property ki_fp_filters "R_*")
 		(sheetname "/")
-		(sheetfile "BYTE_Electronics.kicad_sch")
+		(sheetfile "PDBueno.kicad_sch")
 		(attr smd)
 		(fp_line
@@
 	(footprint "Library_mis componentes:BEC_Matek_12S_Pro"
 		(layer "F.Cu")
-		(at 139.7 93.98)
+		(at 142.24 93.98)
 		(property "Reference" "U1"
 			(at 0 -0.5 0)
@@
 		(property ki_fp_filters "TO?263*")
 		(sheetname "/")
-		(sheetfile "BYTE_Electronics.kicad_sch")
+		(sheetfile "PDBueno.kicad_sch")
 		(attr smd)
 		(fp_rect
@@
 		(property ki_fp_filters "TerminalBlock*:*")
 		(sheetname "/")
-		(sheetfile "BYTE_Electronics.kicad_sch")
+		(sheetfile "PDBueno.kicad_sch")
 		(attr through_hole)
 		(fp_line
@@
 		(layer "Edge.Cuts")
 	)
+	(gr_text "-"
+		(at 114.3 104.14 0)
+		(layer "F.SilkS")
+		(effects
+			(font
+				(size 3 3)
+				(thickness 0.6)
+				(bold yes)
+			)
+			(justify left bottom)
+		)
+	)
+	(gr_text "+"
+		(at 93.48 104.14 0)
+		(layer "F.SilkS")
+		(effects
+			(font
+				(size 3 3)
+				(thickness 0.6)
+				(bold yes)
+			)
+			(justify left bottom)
+		)
+	)
+	(gr_text "-"
+		(at 99.06 104.14 0)
+		(layer "F.SilkS")
+		(effects
+			(font
+				(size 3 3)
+				(thickness 0.6)
+				(bold yes)
+			)
+			(justify left bottom)
+		)
+	)
 	(gr_text "Designed by \n	Anaïs Bueno, Loïc Finette\n	Johnan Luca, Maxime Blanpain"
 		(at 91.44 86.36 0)
@@
 		)
 	)
+	(gr_text "+"
+		(at 109.22 104.14 0)
+		(layer "F.SilkS")
+		(effects
+			(font
+				(size 3 3)
+				(thickness 0.6)
+				(bold yes)
+			)
+			(justify left bottom)
+		)
+	)
+	(segment
+		(start 105.76 68.085)
+		(end 111.76 62.085)
+		(width 0.2)
+		(layer "F.Cu")
+		(net 1)
+	)
+	(segment
+		(start 134.62 55.88)
+		(end 134.62 63.005)
+		(width 0.2)
+		(layer "F.Cu")
+		(net 1)
+	)
+	(segment
+		(start 157.975 68.085)
+		(end 162.56 63.5)
+		(width 0.2)
+		(layer "F.Cu")
+		(net 1)
+	)
+	(segment
+		(start 162.56 63.5)
+		(end 162.56 55.88)
+		(width 0.2)
+		(layer "F.Cu")
+		(net 1)
+	)
+	(segment
+		(start 154.02 68.085)
+		(end 157.975 68.085)
+		(width 0.2)
+		(layer "F.Cu")
+		(net 1)
+	)
 	(segment
 		(start 81.28 101.6)
@@
 	)
 	(segment
+		(start 111.76 62.085)
+		(end 111.76 55.88)
+		(width 0.2)
+		(layer "F.Cu")
+		(net 1)
+	)
+	(segment
 		(start 83.82 104.14)
 		(end 83.82 106.68)
@@
 		(net 1)
 	)
+	(segment
+		(start 134.62 63.005)
+		(end 129.54 68.085)
+		(width 0.2)
+		(layer "F.Cu")
+		(net 1)
+	)
+	(via
+		(at 134.62 55.88)
+		(size 0.6)
+		(drill 0.3)
+		(layers "F.Cu" "B.Cu")
+		(net 1)
+	)
 	(via
 		(at 83.82 106.68)
@@
 	)
 	(via
+		(at 111.76 55.88)
+		(size 0.6)
+		(drill 0.3)
+		(layers "F.Cu" "B.Cu")
+		(net 1)
+	)
+	(via
 		(at 116.84 98.55)
 		(size 0.6)
 		(drill 0.3)
+		(layers "F.Cu" "B.Cu")
+		(net 1)
+	)
+	(via
+		(at 162.56 55.88)
+		(size 0.6)
+		(drill 0.3)

Commit message: 50th copper pour
Parts:
- removed REF** (x4): MountingHole_3.2mm_M3_DIN965, MountingHole:MountingHole_3.2mm_M3_DIN965
- added H1: MountingHole_Pad, MountingHole:MountingHole_3.2mm_M3_Pad_Via, F.Cu at (167.5, 111.8)
- added H2: MountingHole_Pad, MountingHole:MountingHole_3.2mm_M3_Pad_Via, F.Cu at (167.6, 40.5)
- added H3: MountingHole_Pad, MountingHole:MountingHole_3.2mm_M3_Pad_Via, F.Cu at (48.3, 111.8)
- added H4: MountingHole_Pad, MountingHole:MountingHole_3.2mm_M3_Pad_Via, F.Cu at (48.1, 40.6)
- moved C3 5.08 mm to (162.0, 58.6)
- moved J7 4.24 mm to (154.5, 50.8)
- moved R1 2.54 mm to (116.8, 88.4)
- moved C2 2.18 mm to (134.6, 58.6)

Commit message: updates updates updates...
Parts:
- J3, J5: footprint TerminalBlock:TerminalBlock_MaiXu_MX126-5.0-02P_1x02_P5.00mm -> TerminalBlock:TerminalBlock_bornier-2_P5.08mm
Connections:
- J3 pad 1: /+24V -> GND
- J3 pad 2: GND -> /+24V
- J4 pad 1: /+48V -> GND
- J4 pad 2: GND -> /+48V
- J5 pad 1: /+48V -> GND
- J5 pad 2: GND -> /+48V
- J7 pad 1: /+48V -> GND
- J7 pad 2: GND -> /+48V
- J9 pad 1: /+48V -> GND
- J9 pad 2: GND -> /+48V
Routing:
- net /+24V: track 32.0 -> 40.1 mm

Commit message: comment
Other:
- board text added: "Every machine is a smoke machine if used wrong enough"
- board text added: "PDBueno designed by EPFL AI-Team BARK project 16.03.2026"
- board text removed: "Designed by Anaïs Bueno, Loïc Finette Johnan Luca, Maxime Blanpain"
Changed lines of the file:
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@@
 		(tags "terminal block bornier2")
 		(property "Reference" "J3"
-			(at 2.54 -5.08 0)
+			(at 2.54 5.08 0)
 			(layer "F.SilkS")
 			(effects
@@
 		(tags "terminal block bornier2")
 		(property "Reference" "J5"
-			(at 2.54 -5.08 0)
+			(at 2.46 5.08 0)
 			(layer "F.SilkS")
 			(effects
@@
 	)
 	(gr_text "-"
-		(at 114.3 104.14 0)
+		(at 109.3 105.41 0)
 		(layer "F.SilkS")
 		(effects
@@
 		)
 	)
-	(gr_text "Designed by \n	Anaïs Bueno, Loïc Finette\n	Johnan Luca, Maxime Blanpain"
-		(at 88.9 83.82 0)
-		(layer "F.SilkS")
-		(effects
-			(font
-				(size 1 1)
-				(thickness 0.1)
-			)
-			(justify left bottom)
-		)
-	)
-	(gr_text "+"
-		(at 109.22 104.14 0)
+	(gr_text "+\n"
+		(at 114.38 105.41 0)
 		(layer "F.SilkS")
 		(effects
@@
 			)
 			(justify left bottom)
+		)
+	)
+	(gr_text "-"
+		(at 94.06 105.41 0)
+		(layer "F.SilkS")
+		(effects
+			(font
+				(size 3 3)
+				(thickness 0.6)
+				(bold yes)
+			)
+			(justify left bottom)
+		)
+	)
+	(gr_text "PDBueno designed by \n	EPFL AI-Team \n	BARK project\n16.03.2026"
+		(at 96.52 86.36 0)
+		(layer "F.SilkS")
+		(effects
+			(font
+				(size 1 1)
+				(thickness 0.1)
+			)
+			(justify left bottom)
+		)
+	)
+	(gr_text "Every machine\nis a smoke machine\nif used wrong enough"
+		(at 58.42 111.76 0)
+		(layer "F.SilkS")
+		(effects
+			(font
+				(size 1 1)
+				(thickness 0.1)
+			)
+			(justify left bottom)
