File: Good_Boy_Limiter/Good_Boy_Limiter.kicad_pcb (KiCad board)
At the start: 2 copper layers, 90.2 x 96.5 mm, 75 parts, among them CN1 XT30PW-M, CN2 XT30PW-M, J1 UART, J2 Extra General Pins, Q2 AO3422, SW3 RESET1, SW4 BOOT1, U1 ESP32-S3-WROOM-1, U10 B3B-XH-A, U11 B3B-XH-A, U12 B3B-XH-A, U2 TC4427EOA_C636891, U3 LM2576HVR-12, U4 USBLC6-2SC6, U5 SY8120B, U8 B3B-XH-A, U9 LM393DR2G

Commit message: Finished e-scheme
Parts:
- removed C2: 1uF, Capacitor_SMD:C_0805_2012Metric_Pad1.18x1.45mm_HandSolder
- removed L2: SL1050-101M, easyeda2kicad:IND-SMD_L11.5-W10.5
- removed R13: 100, easyeda2kicad:RES-SMD_L6.7-W4.0-LS7.9
- removed U2: TC4427EOA_C636891, easyeda2kicad:SOIC-8_L4.9-W3.9-P1.27-LS6.0-TR
- added C13: 2.2uF, Capacitor_SMD:C_1206_3216Metric, F.Cu at (75.7, 87.6)
- added C14: 2.2uF, Capacitor_SMD:C_1206_3216Metric, F.Cu at (75.7, 91.0)
- added C15: 47uF, easyeda2kicad:CAP-SMD_BD10.0-L10.3-W10.3-LS11.0-R-RD, F.Cu at (88.4, 30.7)
- added Ca1: 3.3nF, Capacitor_SMD:C_0603_1608Metric, F.Cu at (70.9, 79.5)
- added Cb1: 56pF, Capacitor_SMD:C_0603_1608Metric, F.Cu at (70.9, 82.0)
- added Cbst1: 2.2nF, Capacitor_SMD:C_0603_1608Metric, F.Cu at (70.9, 84.5)
- added D10: TVS, Diode_SMD:D_SMB, F.Cu at (43.6, 116.7)
- added D11: SS510C, Diode_SMD:D_SMC, F.Cu at (29.6, 120.1)
- added Dsw1: SS510C, Diode_SMD:D_SMC_Handsoldering, F.Cu at (80.4, 82.1)
- added L3: 22uH, easyeda2kicad:IND-SMD_L11.5-W10.0, F.Cu at (60.6, 83.1)
- added Q1: STB15810, easyeda2kicad:D2PAK_L10.2-W9.0-P5.08-LS16.9-BR, F.Cu at (34.7, 101.9)
- added Q3: NMOS, Package_TO_SOT_SMD:SOT-23, F.Cu at (53.7, 36.8)
- added Q4: AO3400A, easyeda2kicad:SOT-23-3_L2.9-W1.3-P1.90-LS2.4-BR, F.Cu at (54.9, 134.2)
- added R21: 100k, Resistor_SMD:R_0603_1608Metric_Pad0.98x0.95mm_HandSolder, F.Cu at (80.7, 91.5)
- added R22: 453k, Capacitor_SMD:C_0603_1608Metric, F.Cu at (70.9, 87.0)
- added R23: 453k, Capacitor_SMD:C_0603_1608Metric, F.Cu at (70.9, 89.5)
- added R24: 49.9k, Capacitor_SMD:C_0603_1608Metric, F.Cu at (70.9, 92.0)
- added R27: 10k, Resistor_SMD:R_0603_1608Metric_Pad0.98x0.95mm_HandSolder, F.Cu at (37.2, 109.7)
- added R29: 10k, Resistor_SMD:R_0603_1608Metric_Pad0.98x0.95mm_HandSolder, F.Cu at (37.2, 112.2)
- added R30: 10k, Resistor_SMD:R_0603_1608Metric_Pad0.98x0.95mm_HandSolder, F.Cu at (37.2, 114.7)
- added R31: 143k, Resistor_SMD:R_0603_1608Metric_Pad0.98x0.95mm_HandSolder, F.Cu at (37.2, 117.2)
- added R32: 210k, Resistor_SMD:R_0603_1608Metric_Pad0.98x0.95mm_HandSolder, F.Cu at (37.2, 119.8)
- added Rshort1: 0, Resistor_SMD:R_0603_1608Metric_Pad0.98x0.95mm_HandSolder, F.Cu at (37.2, 122.3)
- added Rsns1: 20m, easyeda2kicad:RES-SMD_L6.4-W3.2-1, F.Cu at (44.7, 111.1)
- added TP2: UVLO, TestPoint:TestPoint_Pad_D1.0mm, F.Cu at (48.0, 96.8)
- added TP3: OVLO, TestPoint:TestPoint_Pad_D1.0mm, F.Cu at (48.0, 99.8)
- added U6: 1-178136-3, easyeda2kicad:1-178136-3_TYC, F.Cu at (77.8, 72.7)
- added U7: LM5013DDAR, easyeda2kicad:ESOP-8_L4.9-W3.9-P1.27-LS6.0-BL-EP-1, F.Cu at (84.6, 61.6)
- Cin1: value 100uF -> 100nF; footprint easyeda2kicad:CAP-SMD_BD16.0-L17.0-W17.0-FD -> Capacitor_SMD:C_1206_3216Metric
- Cout1: value 1000uF -> 22uF; footprint easyeda2kicad:CAP-SMD_BD10.0-L10.3-W10.3-FD -> Capacitor_SMD:C_1210_3225Metric
- D2: value SS36 -> SS510C; footprint Diode_SMD:D_SMA_Handsoldering -> Diode_SMD:D_SMC
- R14: value 100 -> 10k; footprint easyeda2kicad:RES-SMD_L6.7-W4.0-LS7.9 -> Resistor_SMD:R_0201_0603Metric_Pad0.64x0.40mm_HandSolder
- R3: value 10 -> 50ohm; footprint LED_SMD:LED_0805_2012Metric_Pad1.15x1.40mm_HandSolder -> easyeda2kicad:RES-TH_BD9.0-L36.5-P40.50-D0.8
- U3: value LM2576HVR-12 -> LM5069MM-2/NOPB; footprint easyeda2kicad:TO-263-5_L10.2-W8.6-P1.70-LS14.4-TL -> easyeda2kicad:VSSOP-10_L3.0-W3.0-P0.50-LS4.9-BL
- moved CN1 154.6 mm to (31.4, 84.2), turned to 0 degrees
- moved H2 151.2 mm to (77.1, 36.9)
- moved Q2 148.6 mm to (41.5, 121.6), turned to 0 degrees
- moved CN2 145.9 mm to (45.9, 84.2), turned to 0 degrees
- moved R3 136.9 mm to (46.5, 72.3)
- moved R14 134.3 mm to (54.2, 137.2), turned to 0 degrees
- moved Cin1 129.9 mm to (45.0, 103.9), turned to 0 degrees
- moved D2 123.7 mm to (29.6, 112.3)
- moved U3 122.3 mm to (44.4, 98.8), turned to 0 degrees
- moved TP9 117.2 mm to (87.9, 46.7)
- moved H3 111.2 mm to (77.1, 44.8)
- moved C10 110.1 mm to (64.7, 118.0), turned to 0 degrees
- moved TP8 106.1 mm to (87.9, 42.6)
- moved C12 93.9 mm to (64.7, 121.5), turned to 0 degrees
- moved H4 92.2 mm to (77.1, 52.8)
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Connections:
- D2 pad 1: Net-(D2-K) -> Net-(D11-A)
- J2 pad 5: /GPIO6 -> unconnected-(J2-Pin_5-Pad5)
- Q2 pad 1: Net-(Q2-G) -> /In-rush controller/GPIO
- Q2 pad 2: +48VOUT -> GND
- Q2 pad 3: /Drain -> Net-(Q2-D)
- R14 pad 1: /Drain -> /3V3
- R14 pad 2: +48VIN -> /GPIO0
- R3 pad 1: Net-(U2-OUTA) -> +48VOUT
- R3 pad 2: Net-(Q2-G) -> /In-rush controller/+48VOUT
- U3 pad 1: +48VIN -> Net-(Q1-D)
- U3 pad 2: Net-(D2-K) -> +48VIN
- U3 pad 3: GND -> Net-(Q2-D)
- U3 pad 4: /+12V -> Net-(U3-OVLO)
- U3 pad 6: GND -> Net-(U3-TIMER)
Routing:
- net /3V3: track 128.1 -> 0.00 mm, vias 4 -> 0
- net GND: track 94.1 -> 0.00 mm, vias 23 -> 0
- net /5VUSB: track 87.8 -> 0.00 mm
- net /+12V: track 73.5 -> 0.00 mm
- net Net-(D8-K): track 67.8 -> 0.00 mm, vias 2 -> 0
- net Net-(D7-K): track 61.6 -> 0.00 mm, vias 2 -> 0
- net /GPIO5: track 55.0 -> 0.00 mm, vias 2 -> 0
- net /GPIO1: track 48.5 -> 0.00 mm
- net /GPIO4: track 47.9 -> 0.00 mm, vias 2 -> 0
- net /GPIO2: track 43.0 -> 0.00 mm
- net +48VOUT: track 42.5 -> 0.00 mm, vias 2 -> 0
- net /D-: track 35.8 -> 0.00 mm
- net /D+: track 34.7 -> 0.00 mm
- net /GPIO3: track 27.0 -> 0.00 mm
- net /GPIO16: track 26.8 -> 0.00 mm
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- removed copper zone on F.Cu, net +48VIN
- removed copper zone on F.Cu, net /3V3
- removed copper zone on F.Cu, net /3V3 Selector/Vin
- removed copper zone on F.Cu, net /Drain
- removed copper zone on B.Cu, net GND
- removed copper zone on F.Cu, net GND
Other:
- board outline removed
- board text removed: "+48VOUT"
- board text removed: "3V3"
- board text removed: "48VIN"
- board text removed: "5VUSB"
- board text removed: "BOOT"
- board text removed: "GND"
- board text removed: "IO15"
- board text removed: "IO16"
- board text removed: "IO6"
- board text removed: "IO7"
- board text removed: "PDB1"
- board text removed: "PDB2"
- board text removed: "PDB3"
- board text removed: "PDB4"
- board text removed: "RESET"
- board text removed: "RX"
- board text removed: "SCL"
- board text removed: "SDA"
- board text removed: "TX"
- board text removed: "V+"

Commit message: started routing
Parts:
- removed D1, D3, D6, D9: 3V3, Package_TO_SOT_SMD:SOT-23
- added Cout2: 220uF, easyeda2kicad:CAP-SMD_BD16.0-L17.0-W17.0-FD, F.Cu at (110.3, 132.8)
- added Ctimer1: 1uF, Capacitor_SMD:C_1206_3216Metric, F.Cu at (101.3, 143.7)
- added D12: BAT54S, Package_TO_SOT_SMD:SOT-23, F.Cu at (144.8, 64.8)
- added D13: BAT54S, Package_TO_SOT_SMD:SOT-23, F.Cu at (157.5, 64.8)
- added D14: BAT54S, Package_TO_SOT_SMD:SOT-23, F.Cu at (166.7, 64.8)
- added D15: BAT54S, Package_TO_SOT_SMD:SOT-23, F.Cu at (179.1, 64.8)
- added R13: 220, Resistor_SMD:R_0603_1608Metric, F.Cu at (100.5, 150.3)
- added R25: 220, Resistor_SMD:R_0603_1608Metric, F.Cu at (106.1, 143.2)
- added R26: 10k, Resistor_SMD:R_0201_0603Metric_Pad0.64x0.40mm_HandSolder, F.Cu at (99.9, 152.4)
- added Rpwr1: 150k, Resistor_SMD:R_0603_1608Metric, F.Cu at (106.1, 145.8)
- TP5: footprint TestPoint:TestPoint_Pad_D2.0mm -> TestPoint:TestPoint_Pad_D1.0mm
- moved R17 125.3 mm to (183.2, 68.6), turned to 180 degrees
- moved R18 122.7 mm to (179.4, 68.6), turned to 180 degrees
- moved R15 111.6 mm to (170.4, 68.6), turned to 180 degrees
- moved R16 109.1 mm to (166.7, 68.6), turned to 180 degrees
- moved R4 99.0 mm to (158.8, 68.6), turned to 180 degrees
- moved R12 96.3 mm to (155.0, 68.6), turned to 180 degrees
- moved C9 83.0 mm to (130.8, 39.4)
- moved R9 81.7 mm to (132.1, 49.5)
- moved Cbs1 79.0 mm to (125.7, 43.2), turned to 90 degrees
- moved R8 77.9 mm to (132.1, 52.1), turned to 180 degrees
- moved C8 74.6 mm to (130.8, 36.8)
- moved U5 73.4 mm to (129.2, 43.1)
- moved L1 72.7 mm to (120.7, 43.6), turned to -90 degrees
- moved TP5 71.9 mm to (113.0, 39.4)
- moved R1 42.7 mm to (141.4, 68.6)
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Connections:
- net Net-(U5-LX) renamed /3V3 Selector/LX
- C1 pad 1: /GPIO1 -> /GPIO10
- C10 pad 1: /GPIO2 -> /GPIO11
- C11 pad 1: /GPIO3 -> /GPIO12
- C12 pad 1: /GPIO4 -> /GPIO13
- C5 pad 1: Net-(U1-EN) -> Net-(U1-TXD0)
- D11 pad 1: /In-rush controller/+48VOUT -> /+12V
- D2 pad 1: Net-(D11-A) -> /In-rush controller/+48VOUT
- Q1 pad 2: Net-(D11-A) -> /In-rush controller/+48VOUT
- Q2 pad 1: /In-rush controller/GPIO -> Net-(Q2-G)
- Q4 pad 3: Net-(Q4-D) -> Net-(D11-A)
- R1 pad 1: GND -> /GPIO10
- R1 pad 2: /GPIO1 -> /Voltage Sensing Modules/V_Sensing1
- R12 pad 1: GND -> /GPIO11
- R12 pad 2: /GPIO2 -> /Voltage Sensing Modules/V_Sensing2
- R15 pad 1: /Voltage Sensing Modules/V_Sensing3 -> GND
- R15 pad 2: /GPIO3 -> /GPIO12
- R16 pad 1: GND -> /GPIO12
- R16 pad 2: /GPIO3 -> /Voltage Sensing Modules/V_Sensing3
- R17 pad 1: /Voltage Sensing Modules/V_Sensing4 -> GND
- R17 pad 2: /GPIO4 -> /GPIO13
- R18 pad 1: GND -> /GPIO13
- R18 pad 2: /GPIO4 -> /Voltage Sensing Modules/V_Sensing4
- R19 pad 1: Net-(U1-USB_D-) -> Net-(U1-IO2)
- R2 pad 1: /Voltage Sensing Modules/V_Sensing1 -> GND
- R2 pad 2: /GPIO1 -> /GPIO10
- R20 pad 1: Net-(U1-USB_D+) -> Net-(U1-IO3)
- R4 pad 1: /Voltage Sensing Modules/V_Sensing2 -> GND
- R4 pad 2: /GPIO2 -> /GPIO11
- R5 pad 2: Net-(U1-EN) -> Net-(U1-TXD0)
- SW3 pad 3: Net-(U1-EN) -> Net-(U1-TXD0)
- SW3 pad 4: Net-(U1-EN) -> Net-(U1-TXD0)
- U1 pad 10: unconnected-(U1-IO17-Pad10) -> /GPIO0
- U1 pad 11: unconnected-(U1-IO18-Pad11) -> /GPIO1
- U1 pad 12: /SDA -> unconnected-(U1-IO8-Pad12)
- U1 pad 13: Net-(U1-USB_D-) -> /GPIO2
- U1 pad 14: Net-(U1-USB_D+) -> /GPIO3
- U1 pad 15: /GPIO3 -> Net-(U1-IO3)
- U1 pad 16: unconnected-(U1-IO46-Pad16) -> /GPIO14
- U1 pad 17: /SCL -> unconnected-(U1-IO9-Pad17)
- U1 pad 23: unconnected-(U1-IO21-Pad23) -> /GPIO4
- U1 pad 24: unconnected-(U1-IO47-Pad24) -> /GPIO15
- U1 pad 25: unconnected-(U1-IO48-Pad25) -> /GPIO16
- U1 pad 26: unconnected-(U1-IO45-Pad26) -> /GPIO13
- U1 pad 27: /GPIO0 -> unconnected-(U1-IO0-Pad27)
- U1 pad 28: unconnected-(U1-IO35-Pad28) -> /GPIO5
- U1 pad 29: unconnected-(U1-IO36-Pad29) -> /GPIO6
- U1 pad 3: Net-(U1-EN) -> /TX
- U1 pad 30: unconnected-(U1-IO37-Pad30) -> /GPIO7
- U1 pad 31: unconnected-(U1-IO38-Pad31) -> /SDA
- U1 pad 32: unconnected-(U1-IO39-Pad32) -> /SCL
- U1 pad 33: unconnected-(U1-IO40-Pad33) -> /GPIO10
- U1 pad 34: unconnected-(U1-IO41-Pad34) -> /GPIO11
- U1 pad 35: unconnected-(U1-IO42-Pad35) -> /GPIO12
- U1 pad 36: /RX -> unconnected-(U1-RXD0-Pad36)
- U1 pad 37: /TX -> Net-(U1-TXD0)
- U1 pad 38: /GPIO2 -> Net-(U1-IO2)
- U1 pad 39: /GPIO1 -> unconnected-(U1-IO1-Pad39)
- U1 pad 4: /GPIO4 -> unconnected-(U1-IO4-Pad4)
- U1 pad 5: /GPIO5 -> unconnected-(U1-IO5-Pad5)
- U1 pad 6: /GPIO6 -> unconnected-(U1-IO6-Pad6)
- U1 pad 7: /GPIO7 -> unconnected-(U1-IO7-Pad7)
- U1 pad 8: /GPIO15 -> unconnected-(U1-IO15-Pad8)
- U1 pad 9: /GPIO16 -> unconnected-(U1-IO16-Pad9)
- U3 pad 9: Net-(D11-A) -> /In-rush controller/+48VOUT
- U6 pad 2: Net-(Q4-D) -> Net-(D11-A)
- U6 pad 4: GND -> (no net)
- U6 pad 5: GND -> (no net)
Routing:
- net /3V3: track 0.00 -> 68.4 mm, vias 0 -> 3
- net /GPIO13: track 0.00 -> 28.4 mm
- net /GPIO10: track 0.00 -> 24.0 mm
- net /GPIO12: track 0.00 -> 16.4 mm
- net /GPIO11: track 0.00 -> 13.7 mm
- net Net-(U5-BS): track 0.00 -> 2.61 mm
- net /3V3 Selector/LX: track 0.00 -> 0.58 mm
- added copper zone on F.Cu, net /3V3 Selector/LX

Commit message: Routing Update
Parts:
- removed D7, D8: LED, LED_SMD:LED_0805_2012Metric_Pad1.15x1.40mm_HandSolder
- removed Q3: NMOS, Package_TO_SOT_SMD:SOT-23
- removed R10, R11: 330, LED_SMD:LED_0805_2012Metric_Pad1.15x1.40mm_HandSolder
- removed U9: LM393DR2G, easyeda2kicad:SOIC-8_L5.0-W4.0-P1.27-LS6.0-BL
- added D16: LED, LED_SMD:LED_0805_2012Metric_Pad1.15x1.40mm_HandSolder, F.Cu at (27.3, 47.3)
- added D17: LED, LED_SMD:LED_0805_2012Metric_Pad1.15x1.40mm_HandSolder, F.Cu at (143.0, 40.8)
- added D18: LED, LED_SMD:LED_0805_2012Metric_Pad1.15x1.40mm_HandSolder, F.Cu at (173.7, 61.0)
- added D9: LED, LED_SMD:LED_0805_2012Metric_Pad1.15x1.40mm_HandSolder, F.Cu at (27.3, 44.3)
- added R28: 4.8K, Resistor_SMD:R_0402_1005Metric, F.Cu at (31.1, 43.7)
- added R33: 1k, Resistor_SMD:R_0402_1005Metric, F.Cu at (31.1, 45.7)
- added R34: 330, Capacitor_SMD:C_0402_1005Metric, F.Cu at (146.2, 40.8)
- added R35: 330, Resistor_SMD:R_0402_1005Metric, F.Cu at (174.2, 64.6)
- C5: footprint Capacitor_SMD:C_0201_0603Metric_Pad0.64x0.40mm_HandSolder -> Capacitor_SMD:C_0402_1005Metric
- R14, R5: footprint Resistor_SMD:R_0201_0603Metric_Pad0.64x0.40mm_HandSolder -> Resistor_SMD:R_0603_1608Metric
- moved R14 132.6 mm to (163.2, 61.7)
- moved L3 113.3 mm to (173.7, 76.1)
- moved C10 112.0 mm to (150.4, 45.8), turned to 90 degrees
- moved C11 111.6 mm to (150.4, 48.3), turned to 90 degrees
- moved C12 111.0 mm to (150.4, 50.9), turned to 90 degrees
- moved D5 104.2 mm to (184.0, 74.0), turned to -90 degrees
- moved Ca1 104.0 mm to (174.9, 83.7), turned to -90 degrees
- moved D4 102.4 mm to (181.5, 67.3), turned to 180 degrees
- moved Cb1 102.2 mm to (172.9, 87.2), turned to -90 degrees
- moved R22 102.1 mm to (172.9, 83.7), turned to 90 degrees
- moved R23 101.8 mm to (172.7, 90.3)
- moved Cout1 99.3 mm to (180.6, 84.4), turned to -90 degrees
- moved R24 98.1 mm to (169.0, 91.1), turned to 90 degrees
- moved Cbst1 96.7 mm to (167.6, 84.3), turned to -90 degrees
- moved C15 92.5 mm to (155.1, 94.8), turned to 90 degrees
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Connections:
- C1 pad 1: /GPIO10 -> /GPIO4
- C10 pad 1: /GPIO11 -> /GPIO6
- C11 pad 1: /GPIO12 -> /GPIO15
- C12 pad 1: /GPIO13 -> /GPIO17
- C5 pad 1: Net-(U1-TXD0) -> Net-(U1-EN)
- D12 pad 3: /GPIO10 -> /GPIO4
- D13 pad 3: /GPIO11 -> /GPIO6
- D14 pad 3: /GPIO12 -> /GPIO15
- D15 pad 3: /GPIO13 -> /GPIO17
- R1 pad 1: /GPIO10 -> /GPIO4
- R12 pad 1: /GPIO11 -> /GPIO6
- R15 pad 2: /GPIO12 -> /GPIO15
- R16 pad 1: /GPIO12 -> /GPIO15
- R17 pad 2: /GPIO13 -> /GPIO17
- R18 pad 1: /GPIO13 -> /GPIO17
- R19 pad 1: Net-(U1-IO2) -> Net-(U1-USB_D-)
- R2 pad 2: /GPIO10 -> /GPIO4
- R20 pad 1: Net-(U1-IO3) -> Net-(U1-USB_D+)
- R4 pad 2: /GPIO11 -> /GPIO6
- R5 pad 2: Net-(U1-TXD0) -> Net-(U1-EN)
- SW3 pad 3: Net-(U1-TXD0) -> Net-(U1-EN)
- SW3 pad 4: Net-(U1-TXD0) -> Net-(U1-EN)
- U1 pad 10: /GPIO0 -> /GPIO17
- U1 pad 11: /GPIO1 -> /GPIO18
- U1 pad 12: unconnected-(U1-IO8-Pad12) -> /SDA
- U1 pad 13: /GPIO2 -> Net-(U1-USB_D-)
- U1 pad 14: /GPIO3 -> Net-(U1-USB_D+)
- U1 pad 15: Net-(U1-IO3) -> /GPIO3
- U1 pad 16: /GPIO14 -> unconnected-(U1-IO46-Pad16)
- U1 pad 17: unconnected-(U1-IO9-Pad17) -> /SCL
- U1 pad 18: unconnected-(U1-IO10-Pad18) -> /GPIO10
- U1 pad 19: unconnected-(U1-IO11-Pad19) -> /GPIO11
- U1 pad 20: unconnected-(U1-IO12-Pad20) -> /GPIO12
- U1 pad 21: unconnected-(U1-IO13-Pad21) -> /GPIO13
- U1 pad 22: unconnected-(U1-IO14-Pad22) -> /GPIO14
- U1 pad 23: /GPIO4 -> unconnected-(U1-IO21-Pad23)
- U1 pad 24: /GPIO15 -> /GPIO47
- U1 pad 25: /GPIO16 -> /GPIO48
- U1 pad 26: /GPIO13 -> unconnected-(U1-IO45-Pad26)
- U1 pad 27: unconnected-(U1-IO0-Pad27) -> /GPIO0
- U1 pad 28: /GPIO5 -> unconnected-(U1-IO35-Pad28)
- U1 pad 29: /GPIO6 -> unconnected-(U1-IO36-Pad29)
- U1 pad 3: /TX -> Net-(U1-EN)
- U1 pad 30: /GPIO7 -> unconnected-(U1-IO37-Pad30)
- U1 pad 31: /SDA -> /GPIO38
- U1 pad 32: /SCL -> /GPIO39
- U1 pad 33: /GPIO10 -> /GPIO40
- U1 pad 34: /GPIO11 -> /GPIO41
- U1 pad 35: /GPIO12 -> /GPIO42
- U1 pad 36: unconnected-(U1-RXD0-Pad36) -> /RX
- U1 pad 37: Net-(U1-TXD0) -> /TX
- U1 pad 38: Net-(U1-IO2) -> /GPIO2
- U1 pad 39: unconnected-(U1-IO1-Pad39) -> /GPIO1
- U1 pad 4: unconnected-(U1-IO4-Pad4) -> /GPIO4
- U1 pad 5: unconnected-(U1-IO5-Pad5) -> /GPIO5
- U1 pad 6: unconnected-(U1-IO6-Pad6) -> /GPIO6
- U1 pad 7: unconnected-(U1-IO7-Pad7) -> /GPIO7
- U1 pad 8: unconnected-(U1-IO15-Pad8) -> /GPIO15
- U1 pad 9: unconnected-(U1-IO16-Pad9) -> /GPIO16
Routing:
- net /5VUSB: track 0.00 -> 85.3 mm, vias 0 -> 2
- net GND: track 0.00 -> 70.3 mm, vias 0 -> 21
- net /D-: track 0.00 -> 53.3 mm
- net /3V3: track 68.4 -> 120.5 mm, vias 3 -> 4
- net /D+: track 0.00 -> 51.9 mm
- net /GPIO17: track 0.00 -> 44.1 mm, vias 0 -> 2
- net /GPIO15: track 0.00 -> 36.0 mm, vias 0 -> 2
- net /+12V: track 0.00 -> 31.8 mm
- net Net-(U1-EN): track 0.00 -> 31.8 mm, vias 0 -> 2
- net /GPIO13: track 28.4 -> 0.53 mm
- net /LinOUT: track 0.00 -> 25.6 mm
- net /GPIO6: track 0.00 -> 24.8 mm, vias 0 -> 2
- net /GPIO10: track 24.0 -> 0.53 mm
- net /GPIO4: track 0.00 -> 18.5 mm, vias 0 -> 2
- net /GPIO0: track 0.00 -> 16.3 mm
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- added copper zone on F.Cu, net +48VIN
- added copper zone on F.Cu, net /3V3
- added copper zone on F.Cu, net /3V3 Selector/Vin
Other:
- board text added: "3V3"
- board text added: "BOOT"
- board text added: "RESET"
