File: Good_Boy_Limiter/Good_Boy_Limiter.kicad_pcb (KiCad board)
At the start: 2 copper layers, 105.4 x 86.5 mm, 106 parts, among them CN1 XT30PW-M, CN2 XT30PW-M, J2 Extra General Pins, Q1 STB15810, Q2 AO3422, Q4 AO3400A, SW3 RESET1, SW4 BOOT1, U1 ESP32-S3-WROOM-1, U10 B3B-XH-A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

Commit message: Added pictures and title page
Parts:
- removed R3: 50ohm, easyeda2kicad:RES-TH_BD9.0-L36.5-P40.50-D0.8
- added Rpre1: 50ohm, easyeda2kicad:RES-TH_BD9.0-L36.5-P40.50-D0.8, F.Cu at (186.6, 114.3)

Commit message: Documentation update
Parts:
- moved C5 19.0 mm to (149.6, 81.5)
- moved L3 19.0 mm to (165.6, 93.2)
- moved Q1 19.0 mm to (201.4, 96.0)
- moved R26 19.0 mm to (187.5, 101.0)
- moved R4 19.0 mm to (128.9, 82.6)
- moved Rpwr1 19.0 mm to (190.0, 90.0)
- moved TP8 19.0 mm to (153.7, 127.6)
- moved C3 19.0 mm to (147.3, 59.2)
- moved CN2 19.0 mm to (200.2, 56.4)
- moved J2 19.0 mm to (179.8, 54.0)
- moved R12 19.0 mm to (128.9, 78.8)
- moved R19 19.0 mm to (141.7, 72.3)
- moved R29 19.0 mm to (187.5, 74.3)
- moved R32 19.0 mm to (190.0, 74.3)
- moved R8 19.0 mm to (170.1, 72.6)
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
Commit message: added 3Ds and added more output fore PDBs
Parts:
- removed CN1: XT30PW-M, easyeda2kicad:CONN-TH_XT30PW-M
- added CN4: XT30UW-F.G.Y, easyeda2kicad:CONN-TH_XT30UW-F.G.Y, F.Cu at (156.2, 130.8)
- added CN5: XT30UW-F.G.Y, easyeda2kicad:CONN-TH_XT30UW-F.G.Y, F.Cu at (148.6, 130.8)
- added CN6: XT30UW-F.G.Y, easyeda2kicad:CONN-TH_XT30UW-F.G.Y, F.Cu at (141.0, 130.8)
- added CN7: XT30UW-F.G.Y, easyeda2kicad:CONN-TH_XT30UW-F.G.Y, F.Cu at (133.3, 130.8)
- R6, R7: moved to B.Cu
- moved Rpre1 13.3 mm to (191.8, 131.4)
- moved TP8 12.4 mm to (165.5, 131.4)
- moved R6 5.50 mm to (133.1, 114.9)
- moved D9 2.05 mm to (161.3, 120.0)
- moved R28 2.05 mm to (161.3, 123.8)
- moved R7 0.73 mm to (133.3, 121.9)
Routing:
- net +48VOUT: track 20.7 -> 5.35 mm
- net GND: track 153.5 -> 144.3 mm, vias 61 -> 56
- net Net-(USB1-CC1): track 9.28 -> 4.68 mm, vias 2 -> 1
- net /In-rush controller/+48VOUT: track 63.3 -> 65.2 mm
- net Net-(USB1-CC2): track 3.94 -> 4.42 mm, vias 0 -> 1
- added copper zone on F.Cu, net +48VOUT

Commit message: Added orange led
Parts:
- added D16: LED, LED_SMD:LED_0805_2012Metric_Pad1.15x1.40mm_HandSolder, F.Cu at (181.0, 86.4)
- added R36: 1.2k, Resistor_SMD:R_0402_1005Metric, F.Cu at (180.3, 89.7)
Routing:
- net /+12V: track 71.4 -> 77.0 mm
- net +48VOUT: track 5.35 -> 8.90 mm
- net GND: track 144.3 -> 147.3 mm
- net Net-(D16-A): track 0.00 -> 2.06 mm

Commit message: Solved DRC and ERC
Parts:
- C3, C4, R6, R7: moved to F.Cu
- U1: footprint RF_Module:ESP32-S3-WROOM-1 -> easyeda2kicad:WIRELM-SMD_ESP32-S3-WROOM-1
- moved C4 9.39 mm to (140.2, 57.7), turned to 90 degrees
- moved C3 5.30 mm to (142.2, 57.7), turned to 90 degrees
- moved D17 4.83 mm to (130.0, 57.9)
- moved R34 4.83 mm to (133.2, 57.9)
- moved U1 3.68 mm to (152.9, 66.0)
Connections:
- R19 pad 2: /D- -> /D-OUT
- R20 pad 2: /D+ -> /D+OUT
- U4 pad 1: /D+ -> /D+OUT
- U4 pad 3: /D- -> /D-OUT
- U4 pad 4: /D- -> /USB Communication/D-IN
- U4 pad 6: /D+ -> /USB Communication/D+IN
- USB1 pad A6: /D+ -> /USB Communication/D+IN
- USB1 pad A7: /D- -> /USB Communication/D-IN
- USB1 pad B6: /D+ -> /USB Communication/D+IN
- USB1 pad B7: /D- -> /USB Communication/D-IN
Routing:
- net /D-: track 58.3 -> 0.00 mm
- net /D+: track 56.9 -> 0.00 mm
- net /D-OUT: track 0.00 -> 51.6 mm
- net /D+OUT: track 0.00 -> 51.2 mm
- net /3V3: track 124.2 -> 133.3 mm
- net /USB Communication/D-IN: track 0.00 -> 6.67 mm
- net GND: track 147.3 -> 141.5 mm, vias 56 -> 66
- net /USB Communication/D+IN: track 0.00 -> 5.68 mm
- net Net-(U5-FB): track 4.16 -> 6.15 mm
- net Net-(USB1-CC1): track 4.68 -> 5.79 mm, vias 1 -> 2
- net Net-(U1-EN): track 32.7 -> 31.6 mm
- net Net-(USB1-CC2): vias 1 -> 0
Other:
- outline, holes or cut-outs redrawn
