File: Good_Boy_Limiter/inrush_controller.kicad_sch (KiCad schematic)
At the start: 19 parts, among them Q1 STB15810, Q2 AO3422, U3 LM5069MM-2/NOPB

Commit message: started routing
Parts:
- Cout2: footprint (none) -> easyeda2kicad:CAP-SMD_BD16.0-L17.0-W17.0-FD
Changed lines of the file:
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@@
 			)
 		)
-		(property "Footprint" ""
+		(property "Footprint" "easyeda2kicad:CAP-SMD_BD16.0-L17.0-W17.0-FD"
 			(at 212.09 64.77 0)
 			(effects

Commit message: Routing Update
Parts:
- Cout2: LCSC Part (none) -> C249883
Changed lines of the file:
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@@
+			)
+		)
+		(property "LCSC Part" "C249883"
+			(at 212.09 64.77 0)
+			(effects
+				(font
+					(size 1.27 1.27)
+				)
+				(hide yes)
 			)
 		)

Commit message: Updated routing
Parts:
- removed R27: 10k, Resistor_SMD:R_0603_1608Metric_Pad0.98x0.95mm_HandSolder, symbol Device:R
Connections:
- net Power_Drain: now reaches Q1.3 (D), Rsns1.1, U3.1 (SEN)
- net GPIO6 renamed GPIO
- no-connect marks 0 -> 1
Changed lines of the file:
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@@
 		(color 0 0 0 0)
 	)
+	(no_connect
+		(at 185.42 71.12)
+	)
 	(wire
 		(pts
@@
 	(wire
 		(pts
-			(xy 185.42 71.12) (xy 193.04 71.12)
-		)
-		(stroke
-			(width 0)
-			(type default)
-		)
-	)
-	(wire
-		(pts
 			(xy 154.94 104.14) (xy 154.94 102.87)
 		)
@@
 	(wire
 		(pts
-			(xy 193.04 71.12) (xy 193.04 67.31)
-		)
-		(stroke
-			(width 0)
-			(type default)
-		)
-	)
-	(wire
-		(pts
 			(xy 116.84 102.87) (xy 102.87 102.87)
 		)
@@
 	(wire
 		(pts
-			(xy 193.04 57.15) (xy 193.04 59.69)
-		)
-		(stroke
-			(width 0)
-			(type default)
-		)
-	)
-	(wire
-		(pts
 			(xy 116.84 81.28) (xy 116.84 82.55)
 		)
@@
 		(pts
 			(xy 191.77 87.63) (xy 203.2 87.63)
+		)
+		(stroke
+			(width 0)
+			(type default)
+		)
+	)
+	(wire
+		(pts
+			(xy 44.45 66.04) (xy 54.61 66.04)
 		)
 		(stroke
@@
 		)
 	)
+	(label "Power_Drain"
+		(at 189.23 87.63 0)
+		(effects
+			(font
+				(size 1.27 1.27)
+			)
+			(justify left bottom)
+		)
+	)
 	(label "+48VOUT"
 		(at 54.61 55.88 180)
@@
 		)
 	)
-	(label "VDD"
-		(at 193.04 57.15 0)
-		(effects
-			(font
-				(size 1.27 1.27)
-			)
-			(justify left bottom)
-		)
-	)
-	(label "GPIO6"
+	(label "GPIO2"
 		(at 121.92 59.69 180)
 		(effects
@@
 			)
 			(justify left bottom)
+		)
+	)
+	(label "GPIO2"
+		(at 54.61 66.04 180)
+		(effects
+			(font
+				(size 1.27 1.27)
+			)
+			(justify right bottom)
 		)
 	)
@@
 		(shape input)
 		(at 44.45 60.96 180)
+		(effects
+			(font
+				(size 1.27 1.27)
+			)
+			(justify right)
+		)
+	)
+	(hierarchical_label "GPIO"
+		(shape input)
+		(at 44.45 66.04 180)
 		(effects
 			(font
@@
 					(unit 1)
 				)
-			)
-		)
-	)
-	(symbol
-		(lib_id "Device:R")
-		(at 193.04 63.5 0)
-		(unit 1)
-		(exclude_from_sim no)
-		(in_bom yes)
-		(on_board yes)
-		(dnp no)
-		(fields_autoplaced yes)
-		(property "Reference" "R27"
-			(at 195.58 62.2299 0)
-			(effects
-				(font
-					(size 1.27 1.27)
-				)
-				(justify left)
-			)
-		)
-		(property "Value" "10k"
-			(at 195.58 64.7699 0)
-			(effects
-				(font
-					(size 1.27 1.27)
-				)
-				(justify left)
-			)
-		)
-		(property "Footprint" "Resistor_SMD:R_0603_1608Metric_Pad0.98x0.95mm_HandSolder"
-			(at 191.262 63.5 90)
-			(effects
-				(font
-					(size 1.27 1.27)
-				)
-				(hide yes)
-			)
-		)
-		(property "Datasheet" "~"
-			(at 193.04 63.5 0)
-			(effects
-				(font
-					(size 1.27 1.27)
-				)
-				(hide yes)
-			)
-		)
-		(property "Description" "Resistor"
-			(at 193.04 63.5 0)
-			(effects
-				(font
-					(size 1.27 1.27)
-				)
-				(hide yes)
-			)
-		)
-		(property "LCSC Part" "C25804"
-			(at 193.04 63.5 0)
-			(effects
-				(font
-					(size 1.27 1.27)
-				)
-				(hide yes)
-			)
-		)
-		(property "Sim.Type" ""
-			(at 193.04 63.5 0)
-			(effects
-				(font
-					(size 1.27 1.27)
-				)
-			)
-		)
-		(pin "2"
-		)
-		(pin "1"
-		)
-		(instances
-			(project ""
-				(path "/e6249df1-5b78-4b75-b804-4c6c30b1afc2/4b6b375c-ae9d-4416-a65c-0698ac0d79e4"
-					(reference "R27")
-					(unit 1)
-				)
