File: Good_Boy_Limiter/inrush_controller.kicad_sch (KiCad schematic)
At the start: 18 parts, among them Q1 STB15810, Q2 AO3422, U3 LM5069MM-2/NOPB

Commit message: Added pictures and title page
Changed lines of the file:
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@@
+	(wire
+		(pts
+			(xy 191.77 86.36) (xy 210.82 86.36)
+		)
+		(stroke
+			(width 0)
+			(type default)
+		)
+	)
 	(wire
 		(pts
@@
 	(wire
 		(pts
-			(xy 214.63 40.64) (xy 214.63 64.77)
+			(xy 214.63 57.15) (xy 214.63 64.77)
 		)
 		(stroke
@@
 		(pts
 			(xy 222.25 64.77) (xy 224.79 64.77)
-		)
-		(stroke
-			(width 0)
-			(type default)
-		)
-	)
-	(wire
-		(pts
-			(xy 191.77 86.36) (xy 210.82 86.36)
 		)
 		(stroke
@@
 	)
 	(label "Power_Drain"
-		(at 196.85 86.36 0)
+		(at 191.77 86.36 0)
 		(effects
 			(font
@@
 	)
 	(label "+48VOUT"
-		(at 214.63 40.64 0)
+		(at 214.63 57.15 0)
 		(effects
 			(font
@@
 		(dnp no)
 		(property "Reference" "R25"
-			(at 121.92 65.532 90)
-			(effects
-				(font
+			(at 121.92 58.928 90)
+			(effects
+				(font
