File: Good_Boy_Limiter/inrush_controller.kicad_sch (KiCad schematic)
At the start: 18 parts, among them Q1 STB15810, Q2 AO3422, U3 LM5069MM-2/NOPB

Commit message: feat: added general power scheme and remouved useless folders
Parts:
- TP2, TP3: now left out of the parts list
Changed lines of the file:
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@@
 		(unit 1)
 		(exclude_from_sim no)
-		(in_bom yes)
+		(in_bom no)
 		(on_board yes)
 		(dnp no)
@@
 		(unit 1)
 		(exclude_from_sim no)
-		(in_bom yes)
-		(on_board yes)
-		(dnp no)
+		(in_bom no)
+		(on_board yes)
+		(dnp no)
