File: Good_Boy_Limiter/USB_communication.kicad_sch (KiCad schematic)
At the start: 8 parts, among them U5 MAX40200AUK+T, U6 AMS1117-3.3

Commit message: Added some footprints
Parts:
- removed Cin3: 10uF, symbol Device:C_Small
- added C7: 22uF, easyeda2kicad:CAP-SMD_BD5.0-L5.3-W5.3-FD, symbol easyeda2kicad:EEEFP1V220AR
- added Cin3: 10uF, easyeda2kicad:C0603, symbol easyeda2kicad:CL10A106MQ8NNNC
- R6, R7: footprint (none) -> LED_SMD:LED_0603_1608Metric_Pad1.05x0.95mm_HandSolder; LCSC Part (none) -> C23186
Connections:
- net +5VUSB: now also Cin3.2
- net GND: now also C7.2, Cin3.1; no longer Cout3.2
- new net: C7.1, Cout3.2
Other:
- note added: "LDO for programming ESP without external source"
- note removed: "LDO for programmi ESP without external source"
Changed lines of the file:
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@@
 		(date "2026-04-17")
 	)
-	(text "LDO for programmi ESP \nwithout external source\n"
+	(text "LDO for programming ESP \nwithout external source\n"
 		(exclude_from_sim no)
-		(at 116.332 31.496 0)
+		(at 116.586 32.766 0)
 		(effects
 			(font
@@
 			)
 		)
-		(property "Footprint" ""
+		(property "Footprint" "LED_SMD:LED_0603_1608Metric_Pad1.05x0.95mm_HandSolder"
 			(at 153.67 117.348 90)
 			(effects
@@
 		)
 		(property "Description" "Resistor"
+			(at 153.67 115.57 0)
+			(effects
+				(font
+					(size 1.27 1.27)
+				)
+				(hide yes)
+			)
+		)
+		(property "LCSC Part" "C23186"
 			(at 153.67 115.57 0)
 			(effects
@@
 	)
 	(symbol
+		(lib_id "easyeda2kicad:CL10A106MQ8NNNC")
+		(at 135.89 57.15 90)
+		(unit 1)
+		(exclude_from_sim no)
+		(in_bom yes)
+		(on_board yes)
+		(dnp no)
+		(fields_autoplaced yes)
+		(property "Reference" "Cin3"
+			(at 139.7 55.8799 90)
+			(effects
+				(font
+					(size 1.27 1.27)
+				)
+				(justify right)
+			)
+		)
+		(property "Value" "10uF"
+			(at 139.7 58.4199 90)
+			(effects
+				(font
+					(size 1.27 1.27)
+				)
+				(justify right)
+			)
+		)
+		(property "Footprint" "easyeda2kicad:C0603"
+			(at 143.51 57.15 0)
+			(effects
+				(font
+					(size 1.27 1.27)
+				)
+				(hide yes)
+			)
+		)
+		(property "Datasheet" "https://lcsc.com/product-detail/Multilayer-Ceramic-Capacitors-MLCC-SMD-SMT_SAMSUNG_CL10A106MQ8NNNC_10uF-106-20-6-3V_C1691.html"
+			(at 146.05 57.15 0)
+			(effects
+				(font
+					(size 1.27 1.27)
+				)
+				(hide yes)
+			)
+		)
+		(property "Description" ""
+			(at 135.89 57.15 0)
+			(effects
+				(font
+					(size 1.27 1.27)
+				)
+				(hide yes)
+			)
+		)
+		(property "Manufacturer" "SAMSUNG(三星)"
+			(at 148.59 57.15 0)
+			(effects
+				(font
+					(size 1.27 1.27)
+				)
+				(hide yes)
+			)
+		)
+		(property "MPN" "CL10A106MQ8NNNC"
+			(at 151.13 57.15 0)
+			(effects
+				(font
+					(size 1.27 1.27)
+				)
+				(hide yes)
+			)
+		)
+		(property "LCSC Part" "C1691"
+			(at 153.67 57.15 0)
+			(effects
+				(font
+					(size 1.27 1.27)
+				)
+				(hide yes)
+			)
+		)
+		(pin "1"
+		)
+		(pin "2"
+		)
+		(instances
+			(project ""
+				(path "/e6249df1-5b78-4b75-b804-4c6c30b1afc2/fdc3caad-3f6e-4f98-8bad-cdd7282ecf49"
+					(reference "Cin3")
+					(unit 1)
+				)
+			)
+		)
+	)
+	(symbol
 		(lib_id "power:GND")
 		(at 124.46 88.9 180)
@@
 	(symbol
 		(lib_id "power:GND")
-		(at 97.79 57.15 0)
+		(at 97.79 68.58 0)
 		(unit 1)
 		(exclude_from_sim no)
@@
 		(fields_autoplaced yes)
 		(property "Reference" "#PWR033"
-			(at 97.79 63.5 0)
+			(at 97.79 74.93 0)
 			(effects
 				(font
@@
 		)
 		(property "Value" "GND"
-			(at 97.79 62.23 0)
+			(at 97.79 73.66 0)
 			(effects
 				(font
@@
 		)
 		(property "Footprint" ""
-			(at 97.79 57.15 0)
+			(at 97.79 68.58 0)
 			(effects
 				(font
@@
 		)
 		(property "Datasheet" ""
-			(at 97.79 57.15 0)
+			(at 97.79 68.58 0)
 			(effects
 				(font
@@
 		)
 		(property "Description" "Power symbol creates a global label with name \"GND\" , ground"
-			(at 97.79 57.15 0)
+			(at 97.79 68.58 0)
 			(effects
 				(font
@@
 			)
 		)
-		(property "Footprint" ""
+		(property "Footprint" "LED_SMD:LED_0603_1608Metric_Pad1.05x0.95mm_HandSolder"
 			(at 100.33 109.728 90)
 			(effects
@@
 		)
 		(property "Description" "Resistor"
+			(at 100.33 107.95 0)
+			(effects
+				(font
+					(size 1.27 1.27)
+				)
+				(hide yes)
+			)
+		)
+		(property "LCSC Part" "C23186"
 			(at 100.33 107.95 0)
 			(effects
@@
 	)
 	(symbol
-		(lib_id "Device:C_Small")
-		(at 135.89 54.61 0)
-		(unit 1)
-		(exclude_from_sim no)
-		(in_bom yes)
-		(on_board yes)
-		(dnp no)
-		(fields_autoplaced yes)
-		(property "Reference" "Cin3"
-			(at 138.43 53.3462 0)
-			(effects
-				(font
-					(size 1.27 1.27)
-				)
-				(justify left)
-			)
-		)
-		(property "Value" "10uF"
-			(at 138.43 55.8862 0)
-			(effects
-				(font
-					(size 1.27 1.27)
-				)
-				(justify left)
-			)
-		)
-		(property "Footprint" ""
-			(at 135.89 54.61 0)
-			(effects
-				(font
-					(size 1.27 1.27)
-				)
-				(hide yes)
-			)
-		)
-		(property "Datasheet" "~"
-			(at 135.89 54.61 0)
-			(effects
-				(font
-					(size 1.27 1.27)
-				)
-				(hide yes)
-			)
-		)
-		(property "Description" "Unpolarized capacitor, small symbol"
-			(at 135.89 54.61 0)
-			(effects
-				(font
-					(size 1.27 1.27)
-				)
-				(hide yes)
-			)
-		)
-		(pin "2"
-		)
-		(pin "1"
-		)
-		(instances
-			(project "Good_Boy_Limiter"
-				(path "/e6249df1-5b78-4b75-b804-4c6c30b1afc2/fdc3caad-3f6e-4f98-8bad-cdd7282ecf49"
-					(reference "Cin3")
-					(unit 1)
-				)
-			)
-		)
-	)
-	(symbol
 		(lib_id "power:GND")
 		(at 115.57 43.18 180)
@@
 	(symbol
 		(lib_id "power:GND")
-		(at 135.89 57.15 0)
+		(at 135.89 62.23 0)
 		(unit 1)
 		(exclude_from_sim no)
@@
 		(fields_autoplaced yes)
 		(property "Reference" "#PWR034"
-			(at 135.89 63.5 0)
+			(at 135.89 68.58 0)
 			(effects
 				(font
@@
 		)
 		(property "Value" "GND"
+			(at 135.89 67.31 0)
+			(effects
+				(font
+					(size 1.27 1.27)
+				)
+			)
+		)
+		(property "Footprint" ""
 			(at 135.89 62.23 0)
 			(effects
@@
 					(size 1.27 1.27)
 				)
-			)
-		)
-		(property "Footprint" ""
-			(at 135.89 57.15 0)
-			(effects
-				(font
-					(size 1.27 1.27)
-				)
 				(hide yes)
 			)
 		)
 		(property "Datasheet" ""
-			(at 135.89 57.15 0)
+			(at 135.89 62.23 0)
 			(effects
 				(font
@@
 		)
 		(property "Description" "Power symbol creates a global label with name \"GND\" , ground"
-			(at 135.89 57.15 0)
+			(at 135.89 62.23 0)
 			(effects
 				(font
@@
 					(unit 1)
 				)
+			)
+		)
+	)
+	(symbol
+		(lib_id "easyeda2kicad:EEEFP1V220AR")
+		(at 97.79 62.23 0)
+		(unit 1)
+		(exclude_from_sim no)
+		(in_bom yes)
+		(on_board yes)
+		(dnp no)
+		(fields_autoplaced yes)
+		(property "Reference" "C7"
+			(at 101.6 60.5799 0)
+			(effects
+				(font
+					(size 1.27 1.27)
+				)
+				(justify left)
+			)
+		)
+		(property "Value" "22uF"
+			(at 101.6 63.1199 0)
+			(effects
+				(font
+					(size 1.27 1.27)
+				)
+				(justify left)
+			)
+		)
+		(property "Footprint" "easyeda2kicad:CAP-SMD_BD5.0-L5.3-W5.3-FD"
+			(at 97.79 74.93 0)
+			(effects
+				(font
+					(size 1.27 1.27)
+				)
+				(hide yes)
+			)
+		)
+		(property "Datasheet" "https://lcsc.com/product-detail/Others_PANASONIC_EEEFP1V220AR_PANASONIC-EEEFP1V220AR_C178580.html"
+			(at 97.79 77.47 0)
+			(effects
+				(font
+					(size 1.27 1.27)
+				)
+				(hide yes)
+			)
+		)
+		(property "Description" ""
+			(at 97.79 62.23 0)
+			(effects
+				(font
+					(size 1.27 1.27)
+				)
+				(hide yes)
+			)
+		)
+		(property "Manufacturer" "PANASONIC(松下)"
+			(at 97.79 80.01 0)
+			(effects
+				(font
+					(size 1.27 1.27)
+				)
+				(hide yes)
+			)
+		)
+		(property "MPN" "EEEFP1V220AR"
+			(at 97.79 82.55 0)
+			(effects
+				(font
+					(size 1.27 1.27)
+				)
+				(hide yes)
+			)
+		)
+		(property "LCSC Part" "C178580"
+			(at 97.79 85.09 0)
+			(effects
+				(font
+					(size 1.27 1.27)
+				)
+				(hide yes)
+			)
+		)
+		(pin "2"
+		)
+		(pin "1"
+		)
+		(instances
+			(project ""
+				(path "/e6249df1-5b78-4b75-b804-4c6c30b1afc2/fdc3caad-3f6e-4f98-8bad-cdd7282ecf49"
+					(reference "C7")
+					(unit 1)
+				)

Commit message: Added all footprints
Parts:
- removed C7: 22uF, easyeda2kicad:CAP-SMD_BD5.0-L5.3-W5.3-FD, symbol easyeda2kicad:EEEFP1V220AR
- removed Cin3: 10uF, easyeda2kicad:C0603, symbol easyeda2kicad:CL10A106MQ8NNNC
- removed Cout3: 22uF, symbol Device:C_Small
- removed D4: 1N4148W, Diode_SMD:D_SOD-123, symbol Diode:1N4148W
- removed U5: MAX40200AUK+T, easyeda2kicad:TSOT-23-5_L2.9-W1.6-P0.95-LS2.8-BL, symbol easyeda2kicad:MAX40200AUK+T
- removed U6: AMS1117-3.3, Package_TO_SOT_SMD:SOT-223-3_TabPin2, symbol Regulator_Linear:AMS1117-3.3
Connections:
- net +5VUSB renamed 5VUSB
- no-connect marks 3 -> 2
Other:
- note removed: "Ideal Diode fo Buck and LDO voltages <-"
- note removed: "LDO for programming ESP without external source"
- moved on the sheet: R6, R7, USB1

Commit message: Routing update
Parts:
- added U4: USBLC6-2SC6, Package_TO_SOT_SMD:SOT-23-6, symbol Power_Protection:USBLC6-2SC6
Connections:
- net 5VUSB: now also U4.5 (VBUS)
- net D+: now also U4.1 (I/O1), U4.6 (I/O1)
- net D-: now also U4.3 (I/O2), U4.4 (I/O2)
- net GND: now also U4.2 (GND)

Commit message: Updated routing
Other:
- note added: "ESD Protection"
Changed lines of the file:
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@@
 		(date "2026-04-17")
+	)
+	(text "ESD Protection\n"
+		(exclude_from_sim no)
+		(at 84.582 124.206 0)
+		(effects
+			(font
+				(size 1.27 1.27)
+			)
+		)
 	)
 	(junction

Commit message: Routing Update
Parts:
- added D18: LED, LED_SMD:LED_0805_2012Metric_Pad1.15x1.40mm_HandSolder, symbol Device:LED
- added R35: 330, Resistor_SMD:R_0402_1005Metric, symbol Device:R
Connections:
- net 5VUSB: now also R35.1
- net GND: now also D18.1 (K)
- new net: D18.2 (A), R35.2

Commit message: Solved DRC and ERC
Connections:
- net D+: no longer U4.6 (I/O1), USB1.A6 (DP1), USB1.B6 (DP2)
- net D-: no longer U4.4 (I/O2), USB1.A7 (DN1), USB1.B7 (DN2)
- new net D+IN: U4.6 (I/O1), USB1.A6 (DP1), USB1.B6 (DP2)
- new net D-IN: U4.4 (I/O2), USB1.A7 (DN1), USB1.B7 (DN2)
Changed lines of the file:
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@@
 	(wire
 		(pts
-			(xy 46.99 66.04) (xy 53.34 66.04)
+			(xy 46.99 66.04) (xy 54.61 66.04)
 		)
 		(stroke
@@
 	(wire
 		(pts
-			(xy 76.2 107.95) (xy 80.01 107.95)
+			(xy 73.66 107.95) (xy 80.01 107.95)
 		)
 		(stroke
@@
 	(wire
 		(pts
-			(xy 46.99 69.85) (xy 53.34 69.85)
+			(xy 46.99 69.85) (xy 54.61 69.85)
 		)
 		(stroke
@@
 	(wire
 		(pts
-			(xy 95.25 107.95) (xy 90.17 107.95)
+			(xy 97.79 107.95) (xy 90.17 107.95)
 		)
 		(stroke
@@
 	(wire
 		(pts
-			(xy 76.2 110.49) (xy 80.01 110.49)
+			(xy 73.66 110.49) (xy 80.01 110.49)
 		)
 		(stroke
@@
 	(wire
 		(pts
-			(xy 95.25 110.49) (xy 90.17 110.49)
-		)
-		(stroke
-			(width 0)
-			(type default)
-		)
-	)
-	(label "D-"
-		(at 95.25 110.49 180)
-		(effects
-			(font
-				(size 1.27 1.27)
-			)
-			(justify right bottom)
-		)
-	)
-	(label "D-"
+			(xy 97.79 110.49) (xy 90.17 110.49)
+		)
+		(stroke
+			(width 0)
+			(type default)
+		)
+	)
+	(label "D+OUT"
+		(at 54.61 66.04 180)
+		(effects
+			(font
+				(size 1.27 1.27)
+			)
+			(justify right bottom)
+		)
+	)
+	(label "D-IN"
+		(at 97.79 110.49 180)
+		(effects
+			(font
+				(size 1.27 1.27)
+			)
+			(justify right bottom)
+		)
+	)
+	(label "+5VUSB"
+		(at 85.09 64.77 0)
+		(effects
+			(font
+				(size 1.27 1.27)
+			)
+			(justify left bottom)
+		)
+	)
+	(label "D+IN"
+		(at 124.46 72.39 180)
+		(effects
+			(font
+				(size 1.27 1.27)
+			)
+			(justify right bottom)
+		)
+	)
+	(label "D+OUT"
+		(at 73.66 107.95 0)
+		(effects
+			(font
+				(size 1.27 1.27)
+			)
+			(justify left bottom)
+		)
+	)
+	(label "D-OUT"
+		(at 54.61 69.85 180)
+		(effects
+			(font
+				(size 1.27 1.27)
+			)
+			(justify right bottom)
+		)
+	)
+	(label "+5VUSB"
+		(at 85.09 97.79 180)
+		(effects
+			(font
+				(size 1.27 1.27)
+			)
+			(justify right bottom)
+		)
+	)
+	(label "+5VUSB"
+		(at 57.15 81.28 180)
+		(effects
+			(font
+				(size 1.27 1.27)
+			)
+			(justify right bottom)
+		)
+	)
+	(label "D-IN"
+		(at 124.46 69.85 180)
+		(effects
+			(font
+				(size 1.27 1.27)
+			)
+			(justify right bottom)
+		)
+	)
+	(label "+5VUSB"
+		(at 127 77.47 180)
+		(effects
+			(font
+				(size 1.27 1.27)
+			)
+			(justify right bottom)
+		)
+	)
+	(label "+5VUSB"
+		(at 127 64.77 180)
+		(effects
+			(font
+				(size 1.27 1.27)
+			)
+			(justify right bottom)
+		)
+	)
+	(label "D+IN"
+		(at 87.63 69.85 0)
+		(effects
+			(font
+				(size 1.27 1.27)
+			)
+			(justify left bottom)
+		)
+	)
+	(label "D+IN"
+		(at 97.79 107.95 180)
+		(effects
+			(font
+				(size 1.27 1.27)
+			)
+			(justify right bottom)
+		)
+	)
+	(label "+5VUSB"
+		(at 85.09 77.47 0)
+		(effects
+			(font
+				(size 1.27 1.27)
+			)
+			(justify left bottom)
+		)
+	)
+	(label "D-OUT"
+		(at 73.66 110.49 0)
+		(effects
+			(font
+				(size 1.27 1.27)
+			)
+			(justify left bottom)
+		)
+	)
+	(label "D-IN"
 		(at 87.63 72.39 0)
 		(effects
@@
 		)
 	)
-	(label "+5VUSB"
-		(at 85.09 64.77 0)
-		(effects
-			(font
-				(size 1.27 1.27)
-			)
-			(justify left bottom)
-		)
-	)
-	(label "D-"
-		(at 53.34 69.85 180)
-		(effects
-			(font
-				(size 1.27 1.27)
-			)
-			(justify right bottom)
-		)
-	)
-	(label "D+"
-		(at 76.2 107.95 0)
-		(effects
-			(font
-				(size 1.27 1.27)
-			)
-			(justify left bottom)
-		)
-	)
-	(label "D+"
-		(at 87.63 69.85 0)
-		(effects
-			(font
-				(size 1.27 1.27)
-			)
-			(justify left bottom)
-		)
-	)
-	(label "D+"
-		(at 124.46 72.39 180)
-		(effects
-			(font
-				(size 1.27 1.27)
-			)
-			(justify right bottom)
-		)
-	)
-	(label "+5VUSB"
-		(at 85.09 97.79 180)
-		(effects
-			(font
-				(size 1.27 1.27)
-			)
-			(justify right bottom)
-		)
-	)
-	(label "+5VUSB"
-		(at 57.15 81.28 180)
-		(effects
-			(font
-				(size 1.27 1.27)
-			)
-			(justify right bottom)
-		)
-	)
-	(label "D+"
-		(at 53.34 66.04 180)
-		(effects
-			(font
-				(size 1.27 1.27)
-			)
-			(justify right bottom)
-		)
-	)
-	(label "+5VUSB"
-		(at 127 77.47 180)
-		(effects
-			(font
-				(size 1.27 1.27)
-			)
-			(justify right bottom)
-		)
-	)
-	(label "+5VUSB"
-		(at 127 64.77 180)
-		(effects
-			(font
-				(size 1.27 1.27)
-			)
-			(justify right bottom)
-		)
-	)
-	(label "D+"
-		(at 95.25 107.95 180)
-		(effects
-			(font
-				(size 1.27 1.27)
-			)
-			(justify right bottom)
-		)
-	)
-	(label "+5VUSB"
-		(at 85.09 77.47 0)
-		(effects
-			(font
-				(size 1.27 1.27)
-			)
-			(justify left bottom)
-		)
-	)
-	(label "D-"
-		(at 76.2 110.49 0)
-		(effects
-			(font
-				(size 1.27 1.27)
-			)
-			(justify left bottom)
-		)
-	)
-	(label "D-"
-		(at 124.46 69.85 180)
-		(effects
-			(font
-				(size 1.27 1.27)
-			)
-			(justify right bottom)
-		)
-	)
